File: Hardware/board_design/M2_edge_b.sch (KiCad schematic (older format))
At the start: 5 parts

Commit message: rescured and remaped symbols
Parts:
- C70, C71, C72, C73: symbol C -> Device:C
- PCB1: symbol M.2-AE -> PicoEVB-rescue:M.2-AE-m2-board
Changed lines of the file:
@@
-EESchema Schematic File Version 2
-LIBS:power
-LIBS:device
-LIBS:transistors
-LIBS:conn
-LIBS:linear
-LIBS:regul
-LIBS:74xx
-LIBS:cmos4000
-LIBS:adc-dac
-LIBS:memory
-LIBS:xilinx
-LIBS:microcontrollers
-LIBS:dsp
-LIBS:microchip
-LIBS:analog_switches
-LIBS:motorola
-LIBS:texas
-LIBS:intel
-LIBS:audio
-LIBS:interface
-LIBS:digital-audio
-LIBS:philips
-LIBS:display
-LIBS:cypress
-LIBS:siliconi
-LIBS:opto
-LIBS:atmel
-LIBS:contrib
-LIBS:valves
-LIBS:Zilog
-LIBS:zetex
-LIBS:Xicor
-LIBS:Worldsemi
-LIBS:wiznet
-LIBS:video
-LIBS:ttl_ieee
-LIBS:transf
-LIBS:switches
-LIBS:supertex
-LIBS:stm32
-LIBS:stm8
-LIBS:silabs
-LIBS:sensors
-LIBS:rfcom
-LIBS:relays
-LIBS:references
-LIBS:pspice
-LIBS:Power_Management
-LIBS:powerint
-LIBS:Oscillators
-LIBS:onsemi
-LIBS:nxp_armmcu
-LIBS:nordicsemi
-LIBS:msp430
-LIBS:motors
-LIBS:motor_drivers
-LIBS:microchip_pic32mcu
-LIBS:microchip_pic18mcu
-LIBS:microchip_pic16mcu
-LIBS:microchip_pic12mcu
-LIBS:microchip_pic10mcu
-LIBS:microchip_dspic33dsc
-LIBS:mechanical
-LIBS:maxim
-LIBS:logo
-LIBS:Lattice
-LIBS:ir
-LIBS:hc11
-LIBS:graphic
-LIBS:gennum
-LIBS:ftdi
-LIBS:ESD_Protection
-LIBS:elec-unifil
-LIBS:diode
-LIBS:dc-dc
-LIBS:cmos_ieee
-LIBS:brooktre
-LIBS:bosch
-LIBS:bbd
-LIBS:battery_management
-LIBS:analog_devices
-LIBS:Altera
-LIBS:allegro
-LIBS:actel
-LIBS:ac-dc
-LIBS:74xgxx
-LIBS:xc7a50t-bga325
-LIBS:MAX1589A
-LIBS:MIC47050
-LIBS:TS3L110
-LIBS:W25Q
-LIBS:93LC46B-SOT23
-LIBS:m2-board
-LIBS:ft2232-fixed
-LIBS:tps82084
-LIBS:PicoEVB-cache
-EELAYER 25 0
+EESchema Schematic File Version 4
+EELAYER 30 0
 EELAYER END
 $Descr A 11000 8500
@@
 $EndDescr
 $Comp
-L GND #PWR054
+L power:GND #PWR054
 U 1 1 58818EBF
 P 5950 3850
@@
 $EndComp
 $Comp
-L +3V3 #PWR055
+L power:+3V3 #PWR055
 U 1 1 58818EC5
 P 4450 3450
@@
 USB_2+
 $Comp
-L M.2-AE PCB1
+L PicoEVB-rescue:M.2-AE-m2-board PCB1
 U 1 1 58818ECE
 P 5300 3900
@@
 Connection ~ 4600 3650
 $Comp
-L GND #PWR056
+L power:GND #PWR056
 U 1 1 58818ED9
 P 4600 4350
@@
 	4600 3200 4450 3200
 $Comp
-L C C72
+L Device:C C72
 U 1 1 594F3242
 P 3950 2950
@@
 $EndComp
 $Comp
-L C C70
+L Device:C C70
 U 1 1 58818F05
 P 3650 2850
@@
 PETX0_2+
 $Comp
-L C C71
+L Device:C C71
 U 1 1 594F3244
 P 3800 2600
@@
 $EndComp
 $Comp
-L C C73
+L Device:C C73
 U 1 1 58818F26
 P 4050 2700
