File: Hardware/board_design/USB_IO_b.sch (KiCad schematic (older format))
At the start: 4 parts, among them U7 FT230XQ

Commit message: rescured and remaped symbols
Parts:
- C67, C68, C69: symbol C -> Device:C
- U7: symbol FT230XQ -> PicoEVB-rescue:FT230XQ-PicoEVB-rescue
Changed lines of the file:
@@
-EESchema Schematic File Version 2
-LIBS:power
-LIBS:device
-LIBS:transistors
-LIBS:conn
-LIBS:linear
-LIBS:regul
-LIBS:74xx
-LIBS:cmos4000
-LIBS:adc-dac
-LIBS:memory
-LIBS:xilinx
-LIBS:microcontrollers
-LIBS:dsp
-LIBS:microchip
-LIBS:analog_switches
-LIBS:motorola
-LIBS:texas
-LIBS:intel
-LIBS:audio
-LIBS:interface
-LIBS:digital-audio
-LIBS:philips
-LIBS:display
-LIBS:cypress
-LIBS:siliconi
-LIBS:opto
-LIBS:atmel
-LIBS:contrib
-LIBS:valves
-LIBS:Zilog
-LIBS:zetex
-LIBS:Xicor
-LIBS:Worldsemi
-LIBS:wiznet
-LIBS:video
-LIBS:ttl_ieee
-LIBS:transf
-LIBS:switches
-LIBS:supertex
-LIBS:stm32
-LIBS:stm8
-LIBS:silabs
-LIBS:sensors
-LIBS:rfcom
-LIBS:relays
-LIBS:references
-LIBS:pspice
-LIBS:Power_Management
-LIBS:powerint
-LIBS:Oscillators
-LIBS:onsemi
-LIBS:nxp_armmcu
-LIBS:nordicsemi
-LIBS:msp430
-LIBS:motors
-LIBS:motor_drivers
-LIBS:microchip_pic32mcu
-LIBS:microchip_pic18mcu
-LIBS:microchip_pic16mcu
-LIBS:microchip_pic12mcu
-LIBS:microchip_pic10mcu
-LIBS:microchip_dspic33dsc
-LIBS:mechanical
-LIBS:maxim
-LIBS:logo
-LIBS:Lattice
-LIBS:ir
-LIBS:hc11
-LIBS:graphic
-LIBS:gennum
-LIBS:ftdi
-LIBS:ESD_Protection
-LIBS:elec-unifil
-LIBS:diode
-LIBS:dc-dc
-LIBS:cmos_ieee
-LIBS:brooktre
-LIBS:bosch
-LIBS:bbd
-LIBS:battery_management
-LIBS:analog_devices
-LIBS:Altera
-LIBS:allegro
-LIBS:actel
-LIBS:ac-dc
-LIBS:74xgxx
-LIBS:xc7a50t-bga325
-LIBS:MAX1589A
-LIBS:MIC47050
-LIBS:TS3L110
-LIBS:W25Q
-LIBS:93LC46B-SOT23
-LIBS:m2-board
-LIBS:ft2232-fixed
-LIBS:tps82084
-LIBS:PicoEVB-cache
-EELAYER 25 0
+EESchema Schematic File Version 4
+EELAYER 30 0
 EELAYER END
 $Descr A 11000 8500
@@
 $EndDescr
 $Comp
-L C C67
+L Device:C C67
 U 1 1 587DA52B
 P 5250 1150
@@
 $EndComp
 $Comp
-L GND #PWR050
+L power:GND #PWR050
 U 1 1 587DA6D2
 P 5600 1150
@@
 $EndComp
 $Comp
-L C C68
+L Device:C C68
 U 1 1 587DA891
 P 5250 1350
@@
 $EndComp
 $Comp
-L C C69
+L Device:C C69
 U 1 1 587DA8D6
 P 5250 1550
@@
 NoConn ~ 5300 2800
 $Comp
-L +3V3 #PWR051
+L power:+3V3 #PWR051
 U 1 1 5881D588
 P 4700 1400
@@
 $EndComp
 $Comp
-L +3V3 #PWR052
+L power:+3V3 #PWR052
 U 1 1 594F3248
 P 3700 2600
@@
 JTAG to FPGA
 $Comp
-L FT230XQ U7
+L PicoEVB-rescue:FT230XQ-PicoEVB-rescue U7
 U 1 1 59323D6A
 P 4600 2400
@@
 Connection ~ 4500 1550
 $Comp
-L GND #PWR053
+L power:GND #PWR053
 U 1 1 593248AC
 P 4600 3200
