File: Hardware/board_design/fpga_pcie_b.sch (KiCad schematic (older format))
At the start: 8 parts, among them J1 RX-, J2 RX+, J3 CLKIN-, J4 CLKIN+, J5 TX+, J6 TX-, U1 XC7AxxT-xCSG325

Commit message: rescured and remaped symbols
Parts:
- J1, J2, J3, J4, J5, J6: symbol CONN_COAXIAL -> PicoEVB-rescue:CONN_COAXIAL-PicoEVB-rescue
- R1: symbol R -> Device:R
- U1: symbol xc7a50tcsg325 -> PicoEVB-rescue:xc7a50tcsg325-xc7a50t-bga325
Changed lines of the file:
@@
-EESchema Schematic File Version 2
-LIBS:power
-LIBS:device
-LIBS:transistors
-LIBS:conn
-LIBS:linear
-LIBS:regul
-LIBS:74xx
-LIBS:cmos4000
-LIBS:adc-dac
-LIBS:memory
-LIBS:xilinx
-LIBS:microcontrollers
-LIBS:dsp
-LIBS:microchip
-LIBS:analog_switches
-LIBS:motorola
-LIBS:texas
-LIBS:intel
-LIBS:audio
-LIBS:interface
-LIBS:digital-audio
-LIBS:philips
-LIBS:display
-LIBS:cypress
-LIBS:siliconi
-LIBS:opto
-LIBS:atmel
-LIBS:contrib
-LIBS:valves
-LIBS:Zilog
-LIBS:zetex
-LIBS:Xicor
-LIBS:Worldsemi
-LIBS:wiznet
-LIBS:video
-LIBS:ttl_ieee
-LIBS:transf
-LIBS:switches
-LIBS:supertex
-LIBS:stm32
-LIBS:stm8
-LIBS:silabs
-LIBS:sensors
-LIBS:rfcom
-LIBS:relays
-LIBS:references
-LIBS:pspice
-LIBS:Power_Management
-LIBS:powerint
-LIBS:Oscillators
-LIBS:onsemi
-LIBS:nxp_armmcu
-LIBS:nordicsemi
-LIBS:msp430
-LIBS:motors
-LIBS:motor_drivers
-LIBS:microchip_pic32mcu
-LIBS:microchip_pic18mcu
-LIBS:microchip_pic16mcu
-LIBS:microchip_pic12mcu
-LIBS:microchip_pic10mcu
-LIBS:microchip_dspic33dsc
-LIBS:mechanical
-LIBS:maxim
-LIBS:logo
-LIBS:Lattice
-LIBS:ir
-LIBS:hc11
-LIBS:graphic
-LIBS:gennum
-LIBS:ftdi
-LIBS:ESD_Protection
-LIBS:elec-unifil
-LIBS:diode
-LIBS:dc-dc
-LIBS:cmos_ieee
-LIBS:brooktre
-LIBS:bosch
-LIBS:bbd
-LIBS:battery_management
-LIBS:analog_devices
-LIBS:Altera
-LIBS:allegro
-LIBS:actel
-LIBS:ac-dc
-LIBS:74xgxx
-LIBS:xc7a50t-bga325
-LIBS:MAX1589A
-LIBS:MIC47050
-LIBS:TS3L110
-LIBS:W25Q
-LIBS:93LC46B-SOT23
-LIBS:m2-board
-LIBS:ft2232-fixed
-LIBS:tps82084
-LIBS:PicoEVB-cache
-EELAYER 25 0
+EESchema Schematic File Version 4
+EELAYER 30 0
 EELAYER END
 $Descr A 11000 8500
@@
 P1V2_MGTAVTT_B
 $Comp
-L R R1
+L Device:R R1
 U 1 1 586D129E
 P 4250 1900
@@
 MGT0_TX_B-
 $Comp
-L GND #PWR016
+L power:GND #PWR016
 U 1 1 58882BD6
 P 4350 2950
@@
 $EndComp
 $Comp
-L xc7a50tcsg325 U1
+L PicoEVB-rescue:xc7a50tcsg325-xc7a50t-bga325 U1
 U 5 1 586A5889
 P 4550 2050
@@
 PCI Express / MGT loopback
 $Comp
-L CONN_COAXIAL J2
+L PicoEVB-rescue:CONN_COAXIAL-PicoEVB-rescue J2
 U 1 1 59EB4CCF
 P 1750 2350
@@
 $EndComp
 $Comp
-L CONN_COAXIAL J6
+L PicoEVB-rescue:CONN_COAXIAL-PicoEVB-rescue J6
 U 1 1 59EB4D49
 P 7400 2100
@@
 $EndComp
 $Comp
-L CONN_COAXIAL J5
+L PicoEVB-rescue:CONN_COAXIAL-PicoEVB-rescue J5
 U 1 1 59EB4D73
 P 7050 2100
@@
 $EndComp
 $Comp
-L CONN_COAXIAL J1
+L PicoEVB-rescue:CONN_COAXIAL-PicoEVB-rescue J1
 U 1 1 59EB4DA0
 P 1250 2350
@@
 	7250 2750 6350 2750
 $Comp
-L CONN_COAXIAL J4
+L PicoEVB-rescue:CONN_COAXIAL-PicoEVB-rescue J4
 U 1 1 59EB4EEE
 P 2850 1850
@@
 $EndComp
 $Comp
-L CONN_COAXIAL J3
+L PicoEVB-rescue:CONN_COAXIAL-PicoEVB-rescue J3
 U 1 1 59EB4FDE
 P 2450 1850
@@
 UMGTCLK_0-
 $Comp
-L GND #PWR017
+L power:GND #PWR017
 U 1 1 59ED3E1B
 P 7050 1900
@@
 $EndComp
 $Comp
-L GND #PWR018
+L power:GND #PWR018
 U 1 1 59ED3E5D
 P 1250 2150
@@
 $EndComp
 $Comp
-L GND #PWR019
+L power:GND #PWR019
 U 1 1 59ED3E80
 P 1750 2150
@@
 $EndComp
 $Comp
-L GND #PWR020
+L power:GND #PWR020
 U 1 1 59ED3EA3
 P 2450 1650
@@
 $EndComp
 $Comp
-L GND #PWR021
+L power:GND #PWR021
 U 1 1 59ED3EC6
 P 2850 1650
@@
 $EndComp
 $Comp
-L GND #PWR022
+L power:GND #PWR022
 U 1 1 59ED3F33
 P 7400 1900
