File: Hardware/board_design/power_b.sch (KiCad schematic (older format))
At the start: 30 parts, among them J10 1P2, J11 1P0, J12 GND, J7 3P3, J8 1P8, J9 1P0, U3 TPS82085SIL, U4 MAX1589AETT100T, U5 MIC47050-1.2YML, U6 TPS82085SIL

Commit message: rescured and remaped symbols
Parts:
- C52, C56, C58, C59, C60, C61, C64: symbol C -> Device:C
- C53, C54, C55, C57, C62, C63, C65, C66: symbol CP -> Device:CP
- J10, J11, J12, J7, J8, J9: symbol TEST_1P -> PicoEVB-rescue:TEST_1P-PicoEVB-rescue
- L1: symbol Ferrite_Bead -> Device:Ferrite_Bead
- R2, R3, R4, R5: symbol R -> Device:R
- U3, U6: symbol TPS82084SIL -> PicoEVB-rescue:TPS82084SIL-tps82084
- U4: symbol MAX1589AETTxxxT -> PicoEVB-rescue:MAX1589AETTxxxT-MAX1589A
- U5: symbol MIC47050 -> PicoEVB-rescue:MIC47050-MIC47050
