File: Hardware/board_design/fpga_pwr_cfg_b.sch (KiCad schematic (older format))
At the start: 53 parts, among them U1 XC7AxxT-xCSG325

Commit message: rescured and remaped symbols
Parts:
- C1, C10, C11, C12, C13, C14, C15, C16, C17, C18, C19, C2, C20, C21, C22, C23, C24, C25, C26, C27, C28, C29, C30, C31, C32, C33, C34, C35, C36, C37, C38, C39, C4, C40, C41, C42, C43, C44, C45, C46, C47, C48, C49, C5, C50, C6, C7, C8, C9: symbol C -> Device:C
- C3: symbol CP -> Device:CP
- D1: symbol LED -> Device:LED
- RN1: symbol R_Pack04 -> Device:R_Pack04
- U1: symbol xc7a50tcsg325 -> PicoEVB-rescue:xc7a50tcsg325-xc7a50t-bga325
